File: powerCurveFollower/powerCurveFollower.kicad_sch (KiCad schematic)
At the start: 4 parts, among them U1 TLC59281DBQ, U2 TLC59281DBQ, U3 TLC59281DBQ, U4 TLC59281DBQ

Commit message: General Changes
Parts:
- added C1, C2, C3, C4, C5, C6, C7, C8: 10uF, symbol Device:C
- added C10: 100n, symbol Device:C
- added C11: 10u, Capacitor_SMD:C_0402_1005Metric_Pad0.74x0.62mm_HandSolder, symbol Device:C
- added C12: 100n, Capacitor_SMD:C_0402_1005Metric_Pad0.74x0.62mm_HandSolder, symbol Device:C
- added C9: 10u, symbol Device:C
- added D1, D10, D100, D101, D102, D103, D104, D105, D106, D107, D108, D109, D11, D110, D111, D112, D113, D114, D115, D116, D117, D118, D119, D12, D120, D121, D122, D123, D124, D125, D126, D127, D128, D13, D14, D15, D16, D17, D18, D19, D2, D20, D21, D22, D23, D24, D25, D26, D27, D28, D29, D3, D30, D31, D32, D33, D34, D35, D36, D37, D38, D39, D4, D40, D41, D42, D43, D44, D45, D46, D47, D48, D49, D5, D50, D51, D52, D53, D54, D55, D56, D57, D58, D59, D6, D60, D61, D62, D63, D64, D65, D66, D67, D68, D69, D7, D70, D71, D72, D73, D74, D75, D76, D77, D78, D79, D8, D80, D81, D82, D83, D84, D85, D86, D87, D88, D89, D9, D90, D91, D92, D93, D94, D95, D96, D97, D98, D99: LED, symbol Device:LED
- added D129: SM712_SOT23, Package_TO_SOT_SMD:SOT-23, symbol Diode:SM712_SOT23
- added J1: UDPI, symbol Connector:Conn_01x03_Pin
- added J2: PowerIn, symbol Connector:Conn_01x02_Pin
- added J4: RS485, Connector_JST:JST_NV_B02P-NV_1x02_P5.00mm_Vertical, symbol Connector:Conn_01x02_Pin
- added PWR1, S1: LED, LED_SMD:LED_0402_1005Metric_Pad0.77x0.64mm_HandSolder, symbol Device:LED
- added R1, R2, R3, R4, R5, R6, R7, R8: 2.5k, symbol Device:R_US
- added R10, R9: 10k, Resistor_SMD:R_0402_1005Metric_Pad0.72x0.64mm_HandSolder, symbol Device:R_US
- added R11, R12: 1K, Resistor_SMD:R_0402_1005Metric_Pad0.72x0.64mm_HandSolder, symbol Device:R_US
- added TP1, TP10, TP2, TP3, TP4, TP5, TP6, TP7, TP8, TP9: MISO TP, symbol Connector:TestPoint
- added U10: THVD1450DR, Package_SON:VSON-8-1EP_3x3mm_P0.65mm_EP1.6x2.4mm, symbol Interface_UART:THVD1450DR
- added U5, U6, U7, U8: TLC59281DBQ, TLC59281DBQ:SOP63P600X175-28N, symbol TLC59281DBQ:TLC59281DBQ
- added U9: ATtiny426-M, Package_DFN_QFN:VQFN-20-1EP_3x3mm_P0.4mm_EP1.7x1.7mm, symbol MCU_Microchip_ATtiny:ATtiny426-M
Connections:
- net GND: now reaches U3.1 (GND)
- net GND: now also U1.1 (GND), U2.1 (GND), U4.1 (GND), C1.2, C10.1, C11.2, C12.2, C2.2, C3.2, C4.2, C5.2, C6.2, C7.2, C8.2, C9.1, D129.3 (common), J1.1 (Pin_1), J2.1 (Pin_1), PWR1.1 (K), R1.2, R10.2, R2.2, R3.2, R4.2, R5.2, R6.2, R7.2, R8.2, S1.1 (K), U10.5 (GND), U5.1 (GND), U6.1 (GND), U7.1 (GND), U8.1 (GND), U9.21 (GND), U9.3 (GND)
- net at U3.10 (OUT5): now also D38.1 (K)
- net at U3.11 (OUT6): now also D39.1 (K)
- net at U3.12 (OUT7): now also D40.1 (K)
- net at U3.13 (OUT8): now also D41.1 (K)
- net at U3.14 (OUT9): now also D42.1 (K)
- net at U3.15 (OUT10): now also D43.1 (K)
- net at U3.16 (OUT11): now also D44.1 (K)
- net at U3.17 (OUT12): now also D45.1 (K)
- net at U3.18 (OUT13): now also D46.1 (K)
- net at U3.19 (OUT14): now also D47.1 (K)
- net at U3.2 (SIN): now also U2.22 (SOUT)
- net at U3.20 (OUT15): now also D48.1 (K)
- net BLANK: now reaches U3.21 (BLANK)
- net BLANK: now also U1.21 (BLANK), U2.21 (BLANK), U4.21 (BLANK), U5.21 (BLANK), U6.21 (BLANK), U7.21 (BLANK), U8.21 (BLANK), U9.10 (PB4)
- net at U3.22 (SOUT): now also U4.2 (SIN)
- net at U3.23 (IREF): now also R3.1
- net +5V: now reaches U3.24 (VCC)
- net +5V: now also U1.24 (VCC), U2.24 (VCC), U4.24 (VCC), C1.1, C10.2, C11.1, C12.1, C2.1, C3.1, C4.1, C5.1, C6.1, C7.1, C8.1, C9.2, D1.2 (A), D10.2 (A), D100.2 (A), D101.2 (A), D102.2 (A), D103.2 (A), D104.2 (A), D105.2 (A), D106.2 (A), D107.2 (A), D108.2 (A), D109.2 (A), D11.2 (A), D110.2 (A), D111.2 (A), D112.2 (A), D113.2 (A), D114.2 (A), D115.2 (A), D116.2 (A), D117.2 (A), D118.2 (A), D119.2 (A), D12.2 (A), D120.2 (A), D121.2 (A), D122.2 (A), D123.2 (A), D124.2 (A), D125.2 (A), D126.2 (A), D127.2 (A), D128.2 (A), D13.2 (A), D14.2 (A), D15.2 (A), D16.2 (A), D17.2 (A), D18.2 (A), D19.2 (A), D2.2 (A), D20.2 (A), D21.2 (A), D22.2 (A), D23.2 (A), D24.2 (A), D25.2 (A), D26.2 (A), D27.2 (A), D28.2 (A), D29.2 (A), D3.2 (A), D30.2 (A), D31.2 (A), D32.2 (A), D33.2 (A), D34.2 (A), D35.2 (A), D36.2 (A), D37.2 (A), D38.2 (A), D39.2 (A), D4.2 (A), D40.2 (A), D41.2 (A), D42.2 (A), D43.2 (A), D44.2 (A), D45.2 (A), D46.2 (A), D47.2 (A), D48.2 (A), D49.2 (A), D5.2 (A), D50.2 (A), D51.2 (A), D52.2 (A), D53.2 (A), D54.2 (A), D55.2 (A), D56.2 (A), D57.2 (A), D58.2 (A), D59.2 (A), D6.2 (A), D60.2 (A), D61.2 (A), D62.2 (A), D63.2 (A), D64.2 (A), D65.2 (A), D66.2 (A), D67.2 (A), D68.2 (A), D69.2 (A), D7.2 (A), D70.2 (A), D71.2 (A), D72.2 (A), D73.2 (A), D74.2 (A), D75.2 (A), D76.2 (A), D77.2 (A), D78.2 (A), D79.2 (A), D8.2 (A), D80.2 (A), D81.2 (A), D82.2 (A), D83.2 (A), D84.2 (A), D85.2 (A), D86.2 (A), D87.2 (A), D88.2 (A), D89.2 (A), D9.2 (A), D90.2 (A), D91.2 (A), D92.2 (A), D93.2 (A), D94.2 (A), D95.2 (A), D96.2 (A), D97.2 (A), D98.2 (A), D99.2 (A), J1.3 (Pin_3), J2.2 (Pin_2), R11.1, R9.1, U10.8 (VCC), U5.24 (VCC), U6.24 (VCC), U7.24 (VCC), U8.24 (VCC), U9.4 (VCC)
- net SCLK: now reaches U3.3 (SCLK)
- net SCLK: now also U1.3 (SCLK), U2.3 (SCLK), U4.3 (SCLK), U5.3 (SCLK), U6.3 (SCLK), U7.3 (SCLK), U8.3 (SCLK), U9.15 (PC0)
- net LAT: now reaches U3.4 (LAT)
- net LAT: now also U1.4 (LAT), U2.4 (LAT), U4.4 (LAT), U5.4 (LAT), U6.4 (LAT), U7.4 (LAT), U8.4 (LAT), U9.18 (PC3)
- net at U3.5 (OUT0): now also D33.1 (K)
- net at U3.6 (OUT1): now also D34.1 (K)
- net at U3.7 (OUT2): now also D35.1 (K)
- net at U3.8 (OUT3): now also D36.1 (K)
- net at U3.9 (OUT4): now also D37.1 (K)
- net at U1.10 (OUT5): now also D6.1 (K)
- net at U1.11 (OUT6): now also D4.1 (K)
- net at U1.12 (OUT7): now also D2.1 (K)
- net at U1.13 (OUT8): now also D1.1 (K)
- net at U1.14 (OUT9): now also D3.1 (K)
- net at U1.15 (OUT10): now also D5.1 (K)
- net at U1.16 (OUT11): now also D8.1 (K)
- net at U1.17 (OUT12): now also D10.1 (K)
- net at U1.18 (OUT13): now also D12.1 (K)
- net at U1.19 (OUT14): now also D15.1 (K)
- net SIN: now reaches U1.2 (SIN)
- net SIN: now also U9.17 (PC2)
- net at U1.20 (OUT15): now also D16.1 (K)
- net at U1.22 (SOUT): now also U2.2 (SIN)
- net at U1.23 (IREF): now also R1.1
- net at U1.5 (OUT0): now also D14.1 (K)
- net at U1.6 (OUT1): now also D13.1 (K)
- net at U1.7 (OUT2): now also D11.1 (K)
- net at U1.8 (OUT3): now also D9.1 (K)
- net at U1.9 (OUT4): now also D7.1 (K)
- net at U4.10 (OUT5): now also D54.1 (K)
- net at U4.11 (OUT6): now also D55.1 (K)
- net at U4.12 (OUT7): now also D56.1 (K)
- net at U4.13 (OUT8): now also D57.1 (K)
- net at U4.14 (OUT9): now also D58.1 (K)
- net at U4.15 (OUT10): now also D59.1 (K)
- net at U4.16 (OUT11): now also D60.1 (K)
- net at U4.17 (OUT12): now also D61.1 (K)
- net at U4.18 (OUT13): now also D62.1 (K)
- net at U4.19 (OUT14): now also D63.1 (K)
- net at U4.20 (OUT15): now also D64.1 (K)
- net at U4.22 (SOUT): now also U5.2 (SIN)
- net at U4.23 (IREF): now also R4.1
- net at U4.5 (OUT0): now also D49.1 (K)
- net at U4.6 (OUT1): now also D50.1 (K)
- net at U4.7 (OUT2): now also D51.1 (K)
- net at U4.8 (OUT3): now also D52.1 (K)
- net at U4.9 (OUT4): now also D53.1 (K)
- net at U2.10 (OUT5): now also D22.1 (K)
- net at U2.11 (OUT6): now also D23.1 (K)
- net at U2.12 (OUT7): now also D24.1 (K)
- net at U2.13 (OUT8): now also D25.1 (K)
- net at U2.14 (OUT9): now also D26.1 (K)
- net at U2.15 (OUT10): now also D27.1 (K)
- net at U2.16 (OUT11): now also D28.1 (K)
- net at U2.17 (OUT12): now also D29.1 (K)
- net at U2.18 (OUT13): now also D30.1 (K)
- net at U2.19 (OUT14): now also D31.1 (K)
- net at U2.20 (OUT15): now also D32.1 (K)
- net at U2.23 (IREF): now also R2.1
- net at U2.5 (OUT0): now also D17.1 (K)
- net at U2.6 (OUT1): now also D18.1 (K)
- net at U2.7 (OUT2): now also D19.1 (K)
- net at U2.8 (OUT3): now also D20.1 (K)
- net at U2.9 (OUT4): now also D21.1 (K)
- new net: D96.1 (K), U6.20 (OUT15)
- new net: R6.1, U6.23 (IREF)
- new net: D77.1 (K), U5.11 (OUT6)
- new net: D123.1 (K), U7.18 (OUT13)
- new net: PWR1.2 (A), R11.2
- new net: R7.1, U7.23 (IREF)
- new net: D85.1 (K), U5.15 (OUT10)
- new net: D125.1 (K), U7.19 (OUT14)
- new net: D75.1 (K), U5.10 (OUT5)
- new net: D79.1 (K), U5.12 (OUT7)
- new net: D81.1 (K), U5.13 (OUT8)
- new net: D83.1 (K), U5.14 (OUT9)
- new net: D87.1 (K), U5.16 (OUT11)
- new net: D89.1 (K), U5.17 (OUT12)
- new net: D91.1 (K), U5.18 (OUT13)
- new net: D93.1 (K), U5.19 (OUT14)
- new net: D95.1 (K), U5.20 (OUT15)
- new net: U5.22 (SOUT), U7.2 (SIN)
- new net: R5.1, U5.23 (IREF)
- new net: D65.1 (K), U5.5 (OUT0)
- new net: D67.1 (K), U5.6 (OUT1)
- new net: D69.1 (K), U5.7 (OUT2)
- new net: D71.1 (K), U5.8 (OUT3)
- new net: D73.1 (K), U5.9 (OUT4)
- new net: TP2.1, U9.2 (PA3)
- new net: D86.1 (K), U6.15 (OUT10)
- new net: D70.1 (K), U6.7 (OUT2)
- new net: D129.1 (A1), J4.2 (Pin_2), U10.6 (A)
- new net: D129.2 (A2), J4.1 (Pin_1), U10.7 (B)
- new net: D104.1 (K), U8.8 (OUT3)
- new net: TP6.1, U9.14 (PB0)
- new net: TP8.1, U9.12 (PB2)
- new net: R8.1, U8.23 (IREF)
- new net: J1.2 (Pin_2), U9.19 (~{RESET}/PA0)
- new net: D120.1 (K), U8.16 (OUT11)
- new net: D124.1 (K), U8.18 (OUT13)
- new net: D121.1 (K), U7.17 (OUT12)
- new net: D68.1 (K), U6.6 (OUT1)
- new net: D108.1 (K), U8.10 (OUT5)
- new net: D110.1 (K), U8.11 (OUT6)
- new net: D112.1 (K), U8.12 (OUT7)
- new net: D114.1 (K), U8.13 (OUT8)
- new net: D116.1 (K), U8.14 (OUT9)
- new net: D118.1 (K), U8.15 (OUT10)
- new net: D122.1 (K), U8.17 (OUT12)
- new net: D126.1 (K), U8.19 (OUT14)
- new net: U6.22 (SOUT), U8.2 (SIN)
- new net: D128.1 (K), U8.20 (OUT15)
- new net: TP1.1, U8.22 (SOUT)
- new net: D98.1 (K), U8.5 (OUT0)
- new net: D100.1 (K), U8.6 (OUT1)
- new net: D102.1 (K), U8.7 (OUT2)
- new net: D106.1 (K), U8.9 (OUT4)
- new net: D88.1 (K), U6.16 (OUT11)
- new net: D94.1 (K), U6.19 (OUT14)
- new net: D103.1 (K), U7.8 (OUT3)
- new net: TP7.1, U9.13 (PB1)
- new net: D82.1 (K), U6.13 (OUT8)
- new net: TP9.1, U9.11 (PB3)
- new net: D84.1 (K), U6.14 (OUT9)
- new net: D113.1 (K), U7.13 (OUT8)
- new net: TP3.1, U9.5 (PA4)
- new net: D92.1 (K), U6.18 (OUT13)
- new net: D109.1 (K), U7.11 (OUT6)
- new net: D74.1 (K), U6.9 (OUT4)
- new net: R12.2, S1.2 (A)
- new net: D119.1 (K), U7.16 (OUT11)
- new net: D97.1 (K), U7.5 (OUT0)
- new net: D99.1 (K), U7.6 (OUT1)
- new net: D72.1 (K), U6.8 (OUT3)
- new net: D90.1 (K), U6.17 (OUT12)
- new net: TP4.1, U9.6 (PA5)
- new net: D66.1 (K), U6.5 (OUT0)
- new net: D78.1 (K), U6.11 (OUT6)
- new net: D107.1 (K), U7.10 (OUT5)
- new net: D111.1 (K), U7.12 (OUT7)
- new net: D76.1 (K), U6.10 (OUT5)
- new net: D80.1 (K), U6.12 (OUT7)
- new net: U6.2 (SIN), U7.22 (SOUT)
- new net: TP10.1, U9.16 (PC1)
- new net: D101.1 (K), U7.7 (OUT2)
- new net: D127.1 (K), U7.20 (OUT15)
- new net: TP5.1, U9.7 (PA6)
- new net: D117.1 (K), U7.15 (OUT10)
- new net: D115.1 (K), U7.14 (OUT9)
- new net: D105.1 (K), U7.9 (OUT4)
- new net D3: R12.1, U9.8 (PA7)
- new net D9: R10.1, R9.2, U10.2 (~{RE}), U10.3 (DE)
- new net RXD2: U10.1 (RO), U9.1 (PA2)
- new net TXD2: U10.4 (DI), U9.20 (PA1)
Other:
- moved on the sheet: U1
